Commit message: fix bugs in rviz , plugins gazebo and URDF file

File: urdf/historia.xacro (robot description, xacro)
@@ -20,15 +20,15 @@
     <inertial>
       <origin
-        xyz="0.055093 0.00038263 0.083393"
-        rpy="0 0 0" />
-      <mass
-        value="61.45" />
-      <inertia
-        ixx="6.7335"
-        ixy="0.00012281"
-        ixz="0.56894"
-        iyy="21.02"
-        iyz="-0.014285"
-        izz="21.189" />
+        xyz="0.054871 0.00038249 0.08412"
+        rpy="0 0 0" />
+      <mass
+        value="61.491" />
+      <inertia
+        ixx="6.7839"
+        ixy="0.00011592"
+        ixz="0.58366"
+        iyy="21.073"
+        iyz="-0.014273"
+        izz="21.196" />
     </inertial>
     <visual>
@@ -290,6 +290,6 @@
       <inertia
         ixx="6.5941E-06"
-        ixy="2.6431E-20"
-        ixz="2.7573E-24"
+        ixy="2.6475E-20"
+        ixz="-2.7573E-24"
         iyy="9.8175E-08"
         iyz="-3.2033E-24"
@@ -348,6 +348,6 @@
       <inertia
         ixx="6.5941E-06"
-        ixy="2.6431E-20"
-        ixz="2.7573E-24"
+        ixy="2.6475E-20"
+        ixz="-2.7573E-24"
         iyy="9.8175E-08"
         iyz="-3.2033E-24"
@@ -456,15 +456,15 @@
     <inertial>
       <origin
-        xyz="0.059799 -0.0013168 1.1692"
+        xyz="-0.015563 0.00050656 -0.0099095"
         rpy="0 0 0" />
       <mass
         value="0.040716" />
       <inertia
-        ixx="3.2796E-05"
-        ixy="3.834E-08"
-        ixz="-2.8496E-06"
+        ixx="3.4077E-05"
+        ixy="3.9139E-08"
+        ixz="-3.218E-07"
         iyy="1.0051E-05"
-        iyz="-9.5815E-09"
-        izz="2.7821E-05" />
+        iyz="5.4791E-09"
+        izz="2.6539E-05" />
     </inertial>
     <visual>
@@ -496,6 +496,6 @@
     type="fixed">
     <origin
-      xyz="0 0 0"
-      rpy="0 0 0" />
+      xyz="0.078809 -0.0018233 1.1721"
+      rpy="0 0.13963 0" />
     <parent
       link="base_link" />
@@ -509,15 +509,15 @@
     <inertial>
       <origin
-        xyz="-0.23976 0.37174 1.1241"
+        xyz="-0.015563 -0.00049343 -0.0099095"
         rpy="0 0 0" />
       <mass
         value="0.040716" />
       <inertia
-        ixx="1.0052E-05"
-        ixy="-1.6285E-08"
-        ixz="8.1977E-08"
-        iyy="3.0506E-05"
-        iyz="-3.7774E-06"
-        izz="3.011E-05" />
+        ixx="3.4077E-05"
+        ixy="3.914E-08"
+        ixz="-3.218E-07"
+        iyy="1.0051E-05"
+        iyz="5.4805E-09"
+        izz="2.6539E-05" />
     </inertial>
     <visual>
@@ -549,6 +549,6 @@
     type="fixed">
     <origin
-      xyz="0 0 0"
-      rpy="0 0 0" />
+      xyz="-0.24289 0.38079 1.1267"
+      rpy="-0.054791 0.46336 1.584" />
     <parent
       link="base_link" />
@@ -562,15 +562,15 @@
     <inertial>
       <origin
-        xyz="-0.23557 -0.37387 1.1233"
+        xyz="-0.015563 0.00050655 -0.0099095"
         rpy="0 0 0" />
       <mass
         value="0.040716" />
       <inertia
-        ixx="1.0052E-05"
-        ixy="-4.4207E-08"
-        ixz="4.1112E-08"
-        iyy="2.9847E-05"
-        iyz="3.7545E-06"
-        izz="3.0769E-05" />
+        ixx="3.4077E-05"
+        ixy="3.9136E-08"
+        ixz="-3.218E-07"
+        iyy="1.0051E-05"
+        iyz="5.4764E-09"
+        izz="2.6539E-05" />
     </inertial>
     <visual>
@@ -602,6 +602,6 @@
     type="fixed">
     <origin
-      xyz="0 0 0"
-      rpy="0 0 0" />
+      xyz="-0.23874 -0.3803 1.1273"
+      rpy="0.053105 0.46353 -1.5874" />
     <parent
       link="base_link" />
@@ -615,15 +615,15 @@
     <inertial>
       <origin
-        xyz="-0.50476 -0.00027997 1.0733"
+        xyz="-0.015563 0.00050656 -0.0099095"
         rpy="0 0 0" />
       <mass
         value="0.040716" />
       <inertia
-        ixx="3.3887E-05"
-        ixy="3.9515E-08"
-        ixz="1.224E-06"
+        ixx="3.4077E-05"
+        ixy="3.9139E-08"
+        ixz="-3.218E-07"
         iyy="1.0051E-05"
-        iyz="-6.6812E-10"
-        izz="2.6729E-05" />
+        iyz="5.4788E-09"
+        izz="2.6539E-05" />
     </inertial>
     <visual>
@@ -655,6 +655,6 @@
     type="fixed">
     <origin
-      xyz="0 0 0"
-      rpy="0 0 0" />
+      xyz="-0.52142 0.00022659 1.0812"
+      rpy="0 0.12217 -3.1416" />
     <parent
       link="base_link" />
@@ -668,15 +668,15 @@
     <inertial>
       <origin
-        xyz="0.069498 -0.0011601 1.1359"
+        xyz="-0.0075 4.4409E-16 -1.3323E-15"
         rpy="0 0 0" />
       <mass
         value="0.0015" />
       <inertia
-        ixx="2.6828E-08"
-        ixy="6.2039E-25"
-        ixz="5.0218E-09"
+        ixx="2.5E-08"
+        ixy="4.7107E-25"
+        ixz="1.8363E-22"
         iyy="4.0625E-08"
-        iyz="-6.8932E-25"
-        izz="3.8797E-08" />
+        iyz="1.1494E-25"
+        izz="4.0625E-08" />
     </inertial>
     <visual>
@@ -708,6 +708,6 @@
     type="fixed">
     <origin
-      xyz="0 0 0"
-      rpy="0 0 0" />
+      xyz="0.076545 -0.0011601 1.1333"
+      rpy="0 0.34907 0" />
     <parent
       link="base_link" />
@@ -721,482 +721,5 @@
     <inertial>
       <origin
-        xyz="1.2534 -1.5685E-05 0.045769"
-        rpy="0 0 0" />
-      <mass
-        value="0.0062273" />
-      <inertia
-        ixx="1.2199E-06"
-        ixy="-1.1399E-10"
-        ixz="-4.2755E-09"
-        iyy="2.3852E-07"
-        iyz="2.1039E-10"
-        izz="1.1947E-06" />
-    </inertial>
-    <visual>
-      <origin
-        xyz="0 0 0"
-        rpy="0 0 0" />
-      <geometry>
-        <mesh
-          filename="package://historia/meshes/front_middle_ultra_link.STL" />
-      </geometry>
-      <material
-        name="">
-        <color
-          rgba="0.79216 0.81961 0.93333 1" />
-      </material>
-    </visual>
-    <collision>
-      <origin
-        xyz="0 0 0"
-        rpy="0 0 0" />
-      <geometry>
-        <mesh
-          filename="package://historia/meshes/front_middle_ultra_link.STL" />
-      </geometry>
-    </collision>
-  </link>
-  <joint
-    name="front_middle_ultra_joint"
-    type="fixed">
-    <origin
-      xyz="0 0 0"
-      rpy="0 0 0" />
-    <parent
-      link="base_link" />
-    <child
-      link="front_middle_ultra_link" />
-    <axis
-      xyz="0 0 0" />
-  </joint>
-  <link
-    name="front_left_ultra_link">
-    <inertial>
-      <origin
-        xyz="1.2509 0.1724 0.04575"
-        rpy="0 0 0" />
-      <mass
-        value="0.0062273" />
-      <inertia
-        ixx="9.8104E-07"
-        ixy="4.1851E-07"
-        ixz="3.5723E-08"
-        iyy="4.8388E-07"
-        iyz="-7.4646E-08"
-        izz="1.1882E-06" />
-    </inertial>
-    <visual>
-      <origin
-        xyz="0 0 0"
-        rpy="0 0 0" />
-      <geometry>
-        <mesh
-          filename="package://historia/meshes/front_left_ultra_link.STL" />
-      </geometry>
-      <material
-        name="">
-        <color
-          rgba="0.79216 0.81961 0.93333 1" />
-      </material>
-    </visual>
-    <collision>
-      <origin
-        xyz="0 0 0"
-        rpy="0 0 0" />
-      <geometry>
-        <mesh
-          filename="package://historia/meshes/front_left_ultra_link.STL" />
-      </geometry>
-    </collision>
-  </link>
-  <joint
-    name="front_left_ultra_joint"
-    type="fixed">
-    <origin
-      xyz="0 0 0"
-      rpy="0 0 0" />
-    <parent
-      link="base_link" />
-    <child
-      link="front_left_ultra_link" />
-    <axis
-      xyz="0 0 0" />
-  </joint>
-  <link
-    name="front_right_ultra_link">
-    <inertial>
-      <origin
-        xyz="1.2552 -0.1649 0.044998"
-        rpy="0 0 0" />
-      <mass
-        value="0.0062273" />
-      <inertia
-        ixx="9.8088E-07"
-        ixy="-4.1858E-07"
-        ixz="3.595E-08"
-        iyy="4.8411E-07"
-        iyz="7.501E-08"
-        izz="1.1881E-06" />
-    </inertial>
-    <visual>
-      <origin
-        xyz="0 0 0"
-        rpy="0 0 0" />
-      <geometry>
-        <mesh
-          filename="package://historia/meshes/front_right_ultra_link.STL" />
-      </geometry>
-      <material
-        name="">
-        <color
-          rgba="0.79216 0.81961 0.93333 1" />
-      </material>
-    </visual>
-    <collision>
-      <origin
-        xyz="0 0 0"
-        rpy="0 0 0" />
-      <geometry>
-        <mesh
-          filename="package://historia/meshes/front_right_ultra_link.STL" />
-      </geometry>
-    </collision>
-  </link>
-  <joint
-    name="front_right_ultra_joint"
-    type="fixed">
-    <origin
-      xyz="0 0 0"
-      rpy="0 0 0" />
-    <parent
-      link="base_link" />
-    <child
-      link="front_right_ultra_link" />
-    <axis
-      xyz="0 0 0" />
-  </joint>
-  <link
-    name="left_corner_ultra_link">
-    <inertial>
-      <origin
-        xyz="0.55346 0.47594 0.042834"
-        rpy="0 0 0" />
-      <mass
-        value="0.0062273" />
-      <inertia
-        ixx="6.3334E-07"
-        ixy="4.7802E-07"
-        ixz="-8.0778E-09"
-        iyy="8.1729E-07"
-        iyz="-9.4053E-09"
-        izz="1.2025E-06" />
-    </inertial>
-    <visual>
-      <origin
-        xyz="0 0 0"
-        rpy="0 0 0" />
-      <geometry>
-        <mesh
-          filename="package://historia/meshes/left_corner_ultra_link.STL" />
-      </geometry>
-      <material
-        name="">
-        <color
-          rgba="0.79216 0.81961 0.93333 1" />
-      </material>
-    </visual>
-    <collision>
-      <origin
-        xyz="0 0 0"
-        rpy="0 0 0" />
-      <geometry>
-        <mesh
-          filename="package://historia/meshes/left_corner_ultra_link.STL" />
-      </geometry>
-    </collision>
-  </link>
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
Commit message: add ackermann steering plugin , rqt_steering has an issue

File: urdf/historia.xacro (robot description, xacro)
@@ -20,15 +20,15 @@
     <inertial>
       <origin
-        xyz="0.054871 0.00038249 0.08412"
-        rpy="0 0 0" />
-      <mass
-        value="61.491" />
-      <inertia
-        ixx="6.7839"
-        ixy="0.00011592"
-        ixz="0.58366"
-        iyy="21.073"
-        iyz="-0.014273"
-        izz="21.196" />
+        xyz="0.0548706683832689 0.000382488154849536 0.0841198429581942"
+        rpy="0 0 0" />
+      <mass
+        value="61.4910296924186" />
+      <inertia
+        ixx="6.78389049097288"
+        ixy="0.000115918559669145"
+        ixz="0.58365880503368"
+        iyy="21.0729581709784"
+        iyz="-0.014273448945033"
+        izz="21.1961147402353" />
     </inertial>
     <visual>
@@ -43,5 +43,5 @@
         name="">
         <color
-          rgba="0.79216 0.81961 0.93333 1" />
+          rgba="0.792156862745098 0.819607843137255 0.933333333333333 1" />
       </material>
     </visual>
@@ -675,5 +675,5 @@
         ixx="2.5E-08"
         ixy="4.7107E-25"
-        ixz="1.8363E-22"
+        ixz="1.8198E-22"
         iyy="4.0625E-08"
         iyz="1.1494E-25"
@@ -1247,3 +1247,109 @@
       xyz="0 0 0" />
   </joint>
+  <link
+    name="rear_wheel">
+    <inertial>
+      <origin
+        xyz="-0.00094232 5.7074E-05 -0.0013048"
+        rpy="0 0 0" />
+      <mass
+        value="0.37589" />
+      <inertia
+        ixx="0.00030881"
+        ixy="9.0382E-07"
+        ixz="1.0964E-05"
+        iyy="0.0004598"
+        iyz="-1.9377E-06"
+        izz="0.00031197" />
+    </inertial>
+    <visual>
+      <origin
+        xyz="0 0 0"
+        rpy="0 0 0" />
+      <geometry>
+        <mesh
+          filename="package://historia/meshes/rear_wheel.STL" />
+      </geometry>
+      <material
+        name="">
+        <color
+          rgba="0.79216 0.81961 0.93333 1" />
+      </material>
+    </visual>
+    <collision>
+      <origin
+        xyz="0 0 0"
+        rpy="0 0 0" />
+      <geometry>
+        <mesh
+          filename="package://historia/meshes/rear_wheel.STL" />
+      </geometry>
+    </collision>
+  </link>
+  <joint
+    name="rear_wheel_joint"
+    type="continuous">
+    <origin
+      xyz="-1.0571 0 0.091"
+      rpy="0 0 0" />
+    <parent
+      link="base_link" />
+    <child
+      link="rear_wheel" />
+    <axis
+      xyz="0 1 0" />
+  </joint>
+  <link
+    name="front_steer">
+    <inertial>
+      <origin
+        xyz="0.0023963 0.00019764 0.025"
+        rpy="0 0 0" />
+      <mass
+        value="0.81548" />
+      <inertia
+        ixx="0.0011707"
+        ixy="-3.559E-19"
+        ixz="0"
+        iyy="0.001295"
+        iyz="-1.5308E-20"
+        izz="0.0011065" />
+    </inertial>
+    <visual>
+      <origin
+        xyz="0 0 0"
+        rpy="0 0 0" />
+      <geometry>
+        <mesh
+          filename="package://historia/meshes/front_steer.STL" />
+      </geometry>
+      <material
+        name="">
+        <color
+          rgba="0.79216 0.81961 0.93333 1" />
+      </material>
+    </visual>
+    <collision>
+      <origin
+        xyz="0 0 0"
+        rpy="0 0 0" />
+      <geometry>
+        <mesh
+          filename="package://historia/meshes/front_steer.STL" />
+      </geometry>
+    </collision>
+  </link>
+  <joint
+    name="front_steer_joint"
+    type="continuous">
+    <origin
+      xyz="1.0431 -0.00019764 0.061"
+      rpy="0 0 0" />
+    <parent
+      link="base_link" />
+    <child
+      link="front_steer" />
+    <axis
+      xyz="0 0 1" />
+  </joint>
 </robot>
